Commit message: Hand facing user

File: src/arm_simulation/urdf/robotic_hand.urdf.xacro (robot description, xacro)
@@ -17,4 +17,19 @@
     <color rgba="0.7 0.5 0.3 1.0"/>
   </material>
+  <!-- Base world link for proper orientation -->
+  <link name="world">
+    <visual>
+      <geometry>
+        <box size="0.001 0.001 0.001"/>
+      </geometry>
+      <material name="hand_material"/>
+      <origin xyz="0 0 0" rpy="0 0 0"/>
+    </visual>
+    <inertial>
+      <mass value="0.001"/>
+      <inertia ixx="0.000001" ixy="0" ixz="0" iyy="0.000001" iyz="0" izz="0.000001"/>
+      <origin xyz="0 0 0" rpy="0 0 0"/>
+    </inertial>
+  </link>
   <!-- Base hand link -->
   <link name="hand_base">
@@ -38,4 +53,10 @@
     </inertial>
   </link>
+  <!-- Joint to orient hand properly (rotate so palm faces camera) -->
+  <joint name="hand_orientation_joint" type="fixed">
+    <parent link="world"/>
+    <child link="hand_base"/>
+    <origin xyz="0 0 0.1" rpy="0 -1.5708 0"/>
+  </joint>
   <!-- Finger macro -->
   <xacro:macro name="finger" params="prefix x_pos y_pos rotation">

Commit message: Improve hand visual appearance and clean up display
Visual Improvements:
- Add realistic skin-tone materials (palm, finger, nail colors)
- Hide TF frame labels, arrows, and axes by default for cleaner view
- Reduce TF marker scale for less visual clutter
- Darker background color for better hand contrast
- Fingertips now use nail material for more realistic appearance

The hand now looks much more lifelike with proper skin tones
and a clean, uncluttered visualization interface.

File: src/arm_simulation/urdf/robotic_hand.urdf.xacro (robot description, xacro)
@@ -12,8 +12,14 @@
   <!-- Materials -->
   <material name="hand_material">
-    <color rgba="0.8 0.6 0.4 1.0"/>
+    <color rgba="0.95 0.87 0.73 1.0"/>  <!-- Skin tone -->
   </material>
   <material name="finger_material">
-    <color rgba="0.7 0.5 0.3 1.0"/>
+    <color rgba="0.92 0.83 0.68 1.0"/>  <!-- Slightly darker skin tone -->
+  </material>
+  <material name="palm_material">
+    <color rgba="0.98 0.90 0.76 1.0"/>  <!-- Palm color -->
+  </material>
+  <material name="nail_material">
+    <color rgba="0.95 0.92 0.88 1.0"/>  <!-- Nail color -->
   </material>
   <!-- Base world link for proper orientation -->
@@ -38,5 +44,5 @@
         <box size="${hand_length} ${hand_width} ${hand_height}"/>
       </geometry>
-      <material name="hand_material"/>
+      <material name="palm_material"/>
       <origin xyz="0 0 0" rpy="0 0 0"/>
     </visual>
@@ -109,5 +115,5 @@
           <box size="${finger_length*0.6} ${finger_width*0.8} ${finger_height*0.8}"/>
         </geometry>
-        <material name="finger_material"/>
+        <material name="nail_material"/>
         <origin xyz="${finger_length*0.3} 0 0" rpy="0 0 0"/>
       </visual>
@@ -179,5 +185,5 @@
           <box size="${thumb_length*0.7} ${thumb_width*0.9} ${finger_height*0.9}"/>
         </geometry>
-        <material name="finger_material"/>
+        <material name="nail_material"/>
         <origin xyz="${thumb_length*0.35} 0 0" rpy="0 0 0"/>
       </visual>

Commit message: Fixed alignement of fingers

File: src/arm_simulation/urdf/robotic_hand.urdf.xacro (robot description, xacro)
@@ -66,5 +66,5 @@
   </joint>
   <!-- Finger macro -->
-  <xacro:macro name="finger" params="prefix x_pos y_pos rotation">
+  <xacro:macro name="finger" params="prefix x_pos y_pos z_pos rotation">
     <!-- Proximal phalanx (base of finger) -->
     <link name="${prefix}_proximal">
@@ -135,5 +135,5 @@
       <parent link="hand_base"/>
       <child link="${prefix}_proximal"/>
-      <origin xyz="${x_pos} ${y_pos} ${hand_height/2 + finger_height/2}" rpy="0 0 ${rotation}"/>
+      <origin xyz="${x_pos} ${y_pos} ${z_pos}" rpy="0 0 ${rotation}"/>
       <axis xyz="0 0 1"/>
       <limit lower="-1.57" upper="1.57" effort="10" velocity="1.0"/>
@@ -157,5 +157,5 @@
   </xacro:macro>
   <!-- Thumb macro (slightly different) -->
-  <xacro:macro name="thumb" params="prefix x_pos y_pos rotation">
+  <xacro:macro name="thumb" params="prefix x_pos y_pos z_pos rotation">
     <!-- Proximal phalanx -->
     <link name="${prefix}_proximal">
@@ -205,5 +205,5 @@
       <parent link="hand_base"/>
       <child link="${prefix}_proximal"/>
-      <origin xyz="${x_pos} ${y_pos} ${hand_height/2 + finger_height/2}" rpy="0 0 ${rotation}"/>
+      <origin xyz="${x_pos} ${y_pos} ${z_pos}" rpy="0 0 ${rotation}"/>
       <axis xyz="0 0 1"/>
       <limit lower="-1.57" upper="1.57" effort="10" velocity="1.0"/>
@@ -219,13 +219,13 @@
   </xacro:macro>
   <!-- Instantiate the fingers -->
-  <!-- Thumb -->
-  <xacro:thumb prefix="thumb" x_pos="-0.02" y_pos="-0.035" rotation="-0.5"/>
-  <!-- Index finger -->
-  <xacro:finger prefix="index" x_pos="0.045" y_pos="-0.025" rotation="0"/>
-  <!-- Middle finger -->
-  <xacro:finger prefix="middle" x_pos="0.05" y_pos="-0.005" rotation="0"/>
-  <!-- Ring finger -->
-  <xacro:finger prefix="ring" x_pos="0.045" y_pos="0.015" rotation="0"/>
-  <!-- Pinky finger -->
-  <xacro:finger prefix="pinky" x_pos="0.035" y_pos="0.03" rotation="0"/>
+  <!-- Thumb (positioned on side of palm) -->
+  <xacro:thumb prefix="thumb" x_pos="0.00" y_pos="-0.030" z_pos="0.0" rotation="-0.7"/>
+  <!-- Index finger (positioned on front edge of palm, top surface) -->
+  <xacro:finger prefix="index" x_pos="0.055" y_pos="-0.030" z_pos="0.0" rotation="0"/>
+  <!-- Middle finger (positioned on front edge of palm, top surface, center) -->
+  <xacro:finger prefix="middle" x_pos="0.058" y_pos="-0.010" z_pos="0.0" rotation="0"/>
+  <!-- Ring finger (positioned on front edge of palm, top surface) -->
+  <xacro:finger prefix="ring" x_pos="0.055" y_pos="0.010" z_pos="0.0" rotation="0"/>
+  <!-- Pinky finger (positioned on front edge of palm, top surface) -->
+  <xacro:finger prefix="pinky" x_pos="0.050" y_pos="0.030" z_pos="0.0" rotation="0"/>
 </robot>

Commit message: Fixed hand

File: src/arm_simulation/urdf/robotic_hand.urdf.xacro (robot description, xacro)
@@ -4,5 +4,5 @@
   <xacro:property name="hand_width" value="0.08" />
   <xacro:property name="hand_length" value="0.12" />
-  <xacro:property name="hand_height" value="0.02" />
+  <xacro:property name="hand_height" value="0.01" />
   <xacro:property name="finger_width" value="0.015" />
   <xacro:property name="finger_length" value="0.03" />
