Commit message: - In DOCKER_SETUP.md updated TroubleShooting section - Modified humanoid_upper_body.urdf.xacro to fix face plate with eyes and mouth positions relative. Also made mouth more red.

File: src/arm_simulation/urdf/humanoid_upper_body.urdf.xacro (robot description, xacro)
@@ -46,5 +46,5 @@
   </material>
   <material name="mouth">
-    <color rgba="0.8 0.3 0.3 1.0"/>  <!-- Red mouth -->
+    <color rgba="0.8 0.1 0.1 1.0"/>  <!-- Red mouth -->
   </material>
   <!-- ==================== WORLD LINK ==================== -->
@@ -130,5 +130,5 @@
       <origin xyz="0 0 0" rpy="0 0 0"/>
     </visual>
-    <!-- Face plate (slightly forward) -->
+    <!-- Face plate (forward in +X) -->
     <visual>
       <geometry>
@@ -136,5 +136,5 @@
       </geometry>
       <material name="skin_face"/>
-      <origin xyz="0 0 ${head_radius - face_depth/2}" rpy="0 0 0"/>
+      <origin xyz="0 0.150 ${head_radius - face_depth/2 - 0.090}" rpy="1.5708 0 0"/>
     </visual>
     <!-- Left eye -->
@@ -144,5 +144,5 @@
       </geometry>
       <material name="eyes"/>
-      <origin xyz="${face_width/4} ${face_height/4} ${head_radius + 0.005}" rpy="0 0 0"/>
+      <origin xyz="${face_width/4} 0.19 ${head_radius + -0.050}" rpy="0 0 0"/>
     </visual>
     <!-- Right eye -->
@@ -152,13 +152,13 @@
       </geometry>
       <material name="eyes"/>
-      <origin xyz="${-face_width/4} ${face_height/4} ${head_radius + 0.005}" rpy="0 0 0"/>
+      <origin xyz="${-face_width/4} 0.19 ${head_radius + -0.050}" rpy="0 0 0"/>
     </visual>
     <!-- Mouth -->
     <visual>
       <geometry>
-        <box size="${face_width/3} 0.015 0.01"/>
+        <box size="${face_width/3} 0.01 0.015"/>
       </geometry>
       <material name="mouth"/>
-      <origin xyz="0 ${-face_height/6} ${head_radius + 0.005}" rpy="0 0 0"/>
+      <origin xyz="0 0.19 ${head_radius - 0.15}" rpy="0 0 0"/>
     </visual>
     <collision>
