Commit message: Fixed urdf erros with joints.

File: src/arm_simulation/urdf/humanoid_robot.urdf.xacro (robot description, xacro)
@@ -177,5 +177,5 @@
        mirror=-1 → right (thumb at +Y, abduction -Z)
        ═══════════════════════════════════════════════════════════════════════ -->
-  <xacro:macro name="hand_assembly" params="side mirror">
+  <xacro:macro name="hand_assembly" params="side mirror orient_yaw:=0">
     <link name="${side}_hand_base">
       <visual><geometry><box size="${hand_length} ${hand_width} ${hand_height}"/></geometry>
@@ -187,10 +187,10 @@
         <origin xyz="0 0 0" rpy="0 0 0"/></inertial>
     </link>
-    <!-- Attach hand to wrist — rpy preserved from dual_hands so hand controller
-         joint angles stay valid. Fingers point in hand's local +X. -->
+    <!-- Attach hand below wrist. rpy="0 1.5708 0" maps hand +X → wrist -Z
+         so fingers point downward (away from arm) in neutral pose. -->
     <joint name="${side}_hand_orient" type="fixed">
       <parent link="${side}_wrist"/>
       <child link="${side}_hand_base"/>
-      <origin xyz="0 0 -0.015" rpy="0 -1.5708 0"/>
+      <origin xyz="0 0 -0.04" rpy="0 1.5708 ${orient_yaw}"/>
     </joint>
     <xacro:thumb  prefix="${side}_thumb"  parent_link="${side}_hand_base"
@@ -283,23 +283,23 @@
       <geometry><sphere radius="0.095"/></geometry>
       <material name="hair_color"/></visual>
-    <!-- Left eye white -->
-    <visual><origin xyz="0.09 0.038 0.14" rpy="0 0 0"/>
+    <!-- Left eye white (robot faces +Y toward viewer) -->
+    <visual><origin xyz="0.038 0.09 0.14" rpy="0 0 0"/>
       <geometry><sphere radius="0.018"/></geometry>
       <material name="eye_white"/></visual>
     <!-- Right eye white -->
-    <visual><origin xyz="0.09 -0.038 0.14" rpy="0 0 0"/>
+    <visual><origin xyz="-0.038 0.09 0.14" rpy="0 0 0"/>
       <geometry><sphere radius="0.018"/></geometry>
       <material name="eye_white"/></visual>
     <!-- Left iris -->
-    <visual><origin xyz="0.108 0.038 0.14" rpy="0 1.5708 0"/>
+    <visual><origin xyz="0.038 0.108 0.14" rpy="-1.5708 0 0"/>
       <geometry><cylinder radius="0.010" length="0.004"/></geometry>
       <material name="eye_iris"/></visual>
     <!-- Right iris -->
-    <visual><origin xyz="0.108 -0.038 0.14" rpy="0 1.5708 0"/>
+    <visual><origin xyz="-0.038 0.108 0.14" rpy="-1.5708 0 0"/>
       <geometry><cylinder radius="0.010" length="0.004"/></geometry>
       <material name="eye_iris"/></visual>
     <!-- Mouth -->
-    <visual><origin xyz="0.107 0 0.085" rpy="0 1.5708 0"/>
-      <geometry><box size="0.004 0.052 0.010"/></geometry>
+    <visual><origin xyz="0 0.107 0.085" rpy="0 0 0"/>
+      <geometry><box size="0.052 0.004 0.010"/></geometry>
       <material name="mouth_red"/></visual>
     <collision><origin xyz="0 0 0.11" rpy="0 0 0"/>
@@ -494,6 +494,6 @@
        HANDS — attach to wrists via macro
        ═══════════════════════════════════════════════════════════════════════ -->
-  <xacro:hand_assembly side="left"  mirror="1"/>
-  <xacro:hand_assembly side="right" mirror="-1"/>
+  <xacro:hand_assembly side="left"  mirror="1"  orient_yaw="3.1416"/>
+  <xacro:hand_assembly side="right" mirror="-1" orient_yaw="0"/>
   <!-- ═══════════════════════════════════════════════════════════════════════
        LEFT LEG  (all joints fixed — standing pose)
@@ -554,14 +554,14 @@
   </joint>
   <link name="left_foot">
-    <visual><origin xyz="0.04 0 -0.03" rpy="0 0 0">
-      </origin>
-      <geometry><box size="0.10 0.09 0.06"/></geometry>
-      <material name="body_dark"/></visual>
-    <collision><origin xyz="0.04 0 -0.03" rpy="0 0 0">
-      </origin>
-      <geometry><box size="0.10 0.09 0.06"/></geometry></collision>
+    <visual><origin xyz="0 0.04 -0.03" rpy="0 0 0">
+      </origin>
+      <geometry><box size="0.09 0.10 0.06"/></geometry>
+      <material name="body_dark"/></visual>
+    <collision><origin xyz="0 0.04 -0.03" rpy="0 0 0">
+      </origin>
+      <geometry><box size="0.09 0.10 0.06"/></geometry></collision>
     <inertial><mass value="1.0"/>
       <inertia ixx="0.003" ixy="0" ixz="0" iyy="0.005" iyz="0" izz="0.005"/>
-      <origin xyz="0.04 0 -0.03" rpy="0 0 0"/></inertial>
+      <origin xyz="0 0.04 -0.03" rpy="0 0 0"/></inertial>
   </link>
   <joint name="left_ankle_pitch" type="fixed">
@@ -622,14 +622,14 @@
   </joint>
   <link name="right_foot">
-    <visual><origin xyz="0.04 0 -0.03" rpy="0 0 0">
-      </origin>
-      <geometry><box size="0.10 0.09 0.06"/></geometry>
-      <material name="body_dark"/></visual>
-    <collision><origin xyz="0.04 0 -0.03" rpy="0 0 0">
-      </origin>
-      <geometry><box size="0.10 0.09 0.06"/></geometry></collision>
+    <visual><origin xyz="0 0.04 -0.03" rpy="0 0 0">
+      </origin>
+      <geometry><box size="0.09 0.10 0.06"/></geometry>
+      <material name="body_dark"/></visual>
+    <collision><origin xyz="0 0.04 -0.03" rpy="0 0 0">
+      </origin>
+      <geometry><box size="0.09 0.10 0.06"/></geometry></collision>
     <inertial><mass value="1.0"/>
       <inertia ixx="0.003" ixy="0" ixz="0" iyy="0.005" iyz="0" izz="0.005"/>
-      <origin xyz="0.04 0 -0.03" rpy="0 0 0"/></inertial>
+      <origin xyz="0 0.04 -0.03" rpy="0 0 0"/></inertial>
   </link>
   <joint name="right_ankle_pitch" type="fixed">

Commit message: Fixed issues with hand

File: src/arm_simulation/urdf/humanoid_robot.urdf.xacro (robot description, xacro)
@@ -192,5 +192,5 @@
       <parent link="${side}_wrist"/>
       <child link="${side}_hand_base"/>
-      <origin xyz="0 0 -0.04" rpy="0 1.5708 ${orient_yaw}"/>
+      <origin xyz="0 0 -0.04" rpy="0 0 ${orient_yaw}"/>
     </joint>
     <xacro:thumb  prefix="${side}_thumb"  parent_link="${side}_hand_base"
@@ -494,6 +494,6 @@
        HANDS — attach to wrists via macro
        ═══════════════════════════════════════════════════════════════════════ -->
-  <xacro:hand_assembly side="left"  mirror="1"  orient_yaw="3.1416"/>
-  <xacro:hand_assembly side="right" mirror="-1" orient_yaw="0"/>
+    <xacro:hand_assembly side="left"  mirror="-1"  orient_yaw="1.5708"/>
+    <xacro:hand_assembly side="right" mirror="1" orient_yaw="1.5708"/>
   <!-- ═══════════════════════════════════════════════════════════════════════
        LEFT LEG  (all joints fixed — standing pose)

Commit message: Robot facing camera

File: src/arm_simulation/urdf/humanoid_robot.urdf.xacro (robot description, xacro)
@@ -225,5 +225,5 @@
   <joint name="world_to_base" type="fixed">
     <parent link="world"/><child link="base_link"/>
-    <origin xyz="0 0 0" rpy="0 0 0"/>
+    <origin xyz="0 0 0" rpy="0 0 -1.5708"/>
   </joint>
   <!-- ─── TORSO ────────────────────────────────────────────────────────── -->

Commit message: Checkpoint

File: src/arm_simulation/urdf/humanoid_robot.urdf.xacro (robot description, xacro)
@@ -27,18 +27,30 @@
   <xacro:property name="thumb_r1" value="0.0075"/>
   <xacro:property name="thumb_r2" value="0.0064"/>
-  <!-- ─── Materials ──────────────────────────────────────────────────────── -->
-  <!-- Body -->
-  <material name="body_skin">  <color rgba="0.85 0.72 0.55 1.0"/> </material>
-  <material name="body_dark">  <color rgba="0.30 0.20 0.15 1.0"/> </material>
-  <material name="hair_color"> <color rgba="0.15 0.10 0.08 1.0"/> </material>
-  <material name="eye_white">  <color rgba="0.95 0.95 0.95 1.0"/> </material>
-  <material name="eye_iris">   <color rgba="0.10 0.30 0.60 1.0"/> </material>
-  <material name="mouth_red">  <color rgba="0.75 0.20 0.15 1.0"/> </material>
-  <!-- Hand skin (same as original) -->
-  <material name="skin_palm">    <color rgba="0.96 0.78 0.62 1.0"/> </material>
-  <material name="skin_finger">  <color rgba="0.93 0.74 0.58 1.0"/> </material>
-  <material name="skin_knuckle"> <color rgba="0.88 0.68 0.52 1.0"/> </material>
-  <material name="skin_tip">     <color rgba="0.97 0.80 0.66 1.0"/> </material>
-  <material name="skin_nail">    <color rgba="1.0  0.75 0.80 0.7"/> </material>
+  <!-- ─── Material colors as xacro properties ─────────────────────────── -->
+  <!-- RViz only applies color when <color> appears inside <visual><material>.
+       Define each RGBA here as a property so every visual can inline it. -->
+  <xacro:property name="c_body_skin"   value="0.85 0.72 0.55 1.0"/>
+  <xacro:property name="c_body_dark"   value="0.30 0.20 0.15 1.0"/>
+  <xacro:property name="c_hair_color"  value="0.15 0.10 0.08 1.0"/>
+  <xacro:property name="c_eye_white"   value="0.95 0.95 0.95 1.0"/>
+  <xacro:property name="c_eye_iris"    value="0.10 0.30 0.60 1.0"/>
+  <xacro:property name="c_mouth_red"   value="0.75 0.20 0.15 1.0"/>
+  <xacro:property name="c_skin_palm"   value="0.96 0.78 0.62 1.0"/>
+  <xacro:property name="c_skin_finger" value="0.93 0.74 0.58 1.0"/>
+  <xacro:property name="c_skin_knuckle" value="0.88 0.68 0.52 1.0"/>
+  <xacro:property name="c_skin_tip"    value="0.97 0.80 0.66 1.0"/>
+  <xacro:property name="c_skin_nail"   value="1.0  0.75 0.80 0.7"/>
+  <!-- ─── Material macros (inline color so RViz picks it up) ───────────── -->
+  <xacro:macro name="m_body_skin">   <material name="body_skin">  <color rgba="${c_body_skin}"/>   </material></xacro:macro>
+  <xacro:macro name="m_body_dark">   <material name="body_dark">  <color rgba="${c_body_dark}"/>   </material></xacro:macro>
+  <xacro:macro name="m_hair_color">  <material name="hair_color"> <color rgba="${c_hair_color}"/>  </material></xacro:macro>
+  <xacro:macro name="m_eye_white">   <material name="eye_white">  <color rgba="${c_eye_white}"/>   </material></xacro:macro>
+  <xacro:macro name="m_eye_iris">    <material name="eye_iris">   <color rgba="${c_eye_iris}"/>    </material></xacro:macro>
+  <xacro:macro name="m_mouth_red">   <material name="mouth_red">  <color rgba="${c_mouth_red}"/>   </material></xacro:macro>
+  <xacro:macro name="m_skin_palm">   <material name="skin_palm">    <color rgba="${c_skin_palm}"/>    </material></xacro:macro>
+  <xacro:macro name="m_skin_finger"> <material name="skin_finger">  <color rgba="${c_skin_finger}"/>  </material></xacro:macro>
+  <xacro:macro name="m_skin_knuckle"><material name="skin_knuckle"> <color rgba="${c_skin_knuckle}"/> </material></xacro:macro>
+  <xacro:macro name="m_skin_tip">    <material name="skin_tip">     <color rgba="${c_skin_tip}"/>     </material></xacro:macro>
+  <xacro:macro name="m_skin_nail">   <material name="skin_nail">    <color rgba="${c_skin_nail}"/>    </material></xacro:macro>
   <!-- ═══════════════════════════════════════════════════════════════════════
        FINGER MACRO  (identical logic to dual_robotic_hands.urdf.xacro)
@@ -47,7 +59,7 @@
     <link name="${prefix}_proximal">
       <visual><geometry><sphere radius="${finger_r0}"/></geometry>
-        <material name="skin_knuckle"/><origin xyz="0 0 0" rpy="0 0 0"/></visual>
+        <xacro:m_skin_knuckle/><origin xyz="0 0 0" rpy="0 0 0"/></visual>
       <visual><geometry><cylinder radius="${finger_r1}" length="${proximal_length}"/></geometry>
-        <material name="skin_finger"/>
+        <xacro:m_skin_finger/>
         <origin xyz="${proximal_length/2} 0 0" rpy="0 1.5708 0"/></visual>
       <collision><geometry><box size="${proximal_length} ${finger_r1*2} ${finger_r1*2}"/></geometry>
@@ -59,7 +71,7 @@
     <link name="${prefix}_middle">
       <visual><geometry><sphere radius="${finger_r1*0.92}"/></geometry>
-        <material name="skin_knuckle"/><origin xyz="0 0 0" rpy="0 0 0"/></visual>
+        <xacro:m_skin_knuckle/><origin xyz="0 0 0" rpy="0 0 0"/></visual>
       <visual><geometry><cylinder radius="${finger_r2}" length="${middle_length}"/></geometry>
-        <material name="skin_finger"/>
+        <xacro:m_skin_finger/>
         <origin xyz="${middle_length/2} 0 0" rpy="0 1.5708 0"/></visual>
       <collision><geometry><box size="${middle_length} ${finger_r2*2} ${finger_r2*2}"/></geometry>
@@ -71,10 +83,10 @@
     <link name="${prefix}_distal">
       <visual><geometry><sphere radius="${finger_r2*0.90}"/></geometry>
-        <material name="skin_knuckle"/><origin xyz="0 0 0" rpy="0 0 0"/></visual>
+        <xacro:m_skin_knuckle/><origin xyz="0 0 0" rpy="0 0 0"/></visual>
       <visual><geometry><cylinder radius="${finger_r3}" length="${distal_length}"/></geometry>
-        <material name="skin_finger"/>
+        <xacro:m_skin_finger/>
         <origin xyz="${distal_length/2} 0 0" rpy="0 1.5708 0"/></visual>
       <visual><geometry><sphere radius="${finger_r3*1.1}"/></geometry>
-        <material name="skin_tip"/>
+        <xacro:m_skin_tip/>
         <origin xyz="${distal_length} 0 0" rpy="0 0 0"/></visual>
       <collision><geometry><box size="${distal_length} ${finger_r3*2} ${finger_r3*2}"/></geometry>
@@ -87,5 +99,5 @@
       <visual>
         <geometry><box size="${distal_length*0.75} ${finger_r3*1.8} ${finger_r3*0.6}"/></geometry>
-        <material name="skin_nail"/><origin xyz="0 0 0" rpy="0 0 0"/></visual>
+        <xacro:m_skin_nail/><origin xyz="0 0 0" rpy="0 0 0"/></visual>
       <inertial><mass value="0.001"/>
         <inertia ixx="0.000001" ixy="0" ixz="0" iyy="0.000001" iyz="0" izz="0.000001"/>
@@ -121,7 +133,7 @@
     <link name="${prefix}_proximal">
       <visual><geometry><sphere radius="${thumb_r0}"/></geometry>
-        <material name="skin_knuckle"/><origin xyz="0 0 0" rpy="0 0 0"/></visual>
+        <xacro:m_skin_knuckle/><origin xyz="0 0 0" rpy="0 0 0"/></visual>
       <visual><geometry><cylinder radius="${thumb_r1}" length="${thumb_proximal_length}"/></geometry>
-        <material name="skin_finger"/>
+        <xacro:m_skin_finger/>
         <origin xyz="${thumb_proximal_length/2} 0 0" rpy="0 1.5708 0"/></visual>
       <collision><geometry><box size="${thumb_proximal_length} ${thumb_r1*2} ${thumb_r1*2}"/></geometry>
@@ -133,10 +145,10 @@
     <link name="${prefix}_distal">
       <visual><geometry><sphere radius="${thumb_r1*0.90}"/></geometry>
-        <material name="skin_knuckle"/><origin xyz="0 0 0" rpy="0 0 0"/></visual>
+        <xacro:m_skin_knuckle/><origin xyz="0 0 0" rpy="0 0 0"/></visual>
       <visual><geometry><cylinder radius="${thumb_r2}" length="${thumb_distal_length}"/></geometry>
-        <material name="skin_finger"/>
+        <xacro:m_skin_finger/>
         <origin xyz="${thumb_distal_length/2} 0 0" rpy="0 1.5708 0"/></visual>
       <visual><geometry><sphere radius="${thumb_r2*1.15}"/></geometry>
-        <material name="skin_tip"/>
+        <xacro:m_skin_tip/>
         <origin xyz="${thumb_distal_length} 0 0" rpy="0 0 0"/></visual>
       <collision><geometry><box size="${thumb_distal_length} ${thumb_r2*2} ${thumb_r2*2}"/></geometry>
@@ -149,5 +161,5 @@
       <visual>
         <geometry><box size="${thumb_distal_length*0.75} ${thumb_r2*2.0} ${thumb_r2*0.6}"/></geometry>
-        <material name="skin_nail"/><origin xyz="0 0 0" rpy="0 0 0"/></visual>
+        <xacro:m_skin_nail/><origin xyz="0 0 0" rpy="0 0 0"/></visual>
       <inertial><mass value="0.001"/>
         <inertia ixx="0.000001" ixy="0" ixz="0" iyy="0.000001" iyz="0" izz="0.000001"/>
@@ -180,5 +192,5 @@
     <link name="${side}_hand_base">
       <visual><geometry><box size="${hand_length} ${hand_width} ${hand_height}"/></geometry>
-        <material name="skin_palm"/><origin xyz="0 0 0" rpy="0 0 0"/></visual>
+        <xacro:m_skin_palm/><origin xyz="0 0 0" rpy="0 0 0"/></visual>
       <collision><geometry><box size="${hand_length} ${hand_width} ${hand_height}"/></geometry>
         <origin xyz="0 0 0" rpy="0 0 0"/></collision>
@@ -233,9 +245,9 @@
     <visual><origin xyz="0 0 0.22" rpy="0 0 0"/>
       <geometry><cylinder radius="0.15" length="0.44"/></geometry>
-      <material name="body_dark"/></visual>
+      <xacro:m_body_dark/></visual>
     <!-- Collar bone / chest highlight -->
     <visual><origin xyz="0 0 0.44" rpy="0 0 0"/>
       <geometry><box size="0.28 0.06 0.02"/></geometry>
-      <material name="body_skin"/></visual>
+      <xacro:m_body_skin/></visual>
     <collision><origin xyz="0 0 0.22" rpy="0 0 0"/>
       <geometry><cylinder radius="0.15" length="0.44"/></geometry></collision>
@@ -261,5 +273,5 @@
     <visual><origin xyz="0 0 0.05" rpy="0 0 0"/>
       <geometry><cylinder radius="0.045" length="0.10"/></geometry>
-      <material name="body_skin"/></visual>
+      <xacro:m_body_skin/></visual>
     <collision><origin xyz="0 0 0.05" rpy="0 0 0"/>
       <geometry><cylinder radius="0.045" length="0.10"/></geometry></collision>
@@ -278,29 +290,29 @@
     <visual><origin xyz="0 0 0.11" rpy="0 0 0"/>
       <geometry><sphere radius="0.11"/></geometry>
-      <material name="body_skin"/></visual>
+      <xacro:m_body_skin/></visual>
     <!-- Hair cap (slightly larger sphere, darker) -->
     <visual><origin xyz="0 0 0.16" rpy="0 0 0"/>
       <geometry><sphere radius="0.095"/></geometry>
-      <material name="hair_color"/></visual>
+      <xacro:m_hair_color/></visual>
     <!-- Left eye white (robot faces +Y toward viewer) -->
     <visual><origin xyz="0.038 0.09 0.14" rpy="0 0 0"/>
       <geometry><sphere radius="0.018"/></geometry>
-      <material name="eye_white"/></visual>
+      <xacro:m_eye_white/></visual>
     <!-- Right eye white -->
     <visual><origin xyz="-0.038 0.09 0.14" rpy="0 0 0"/>
       <geometry><sphere radius="0.018"/></geometry>
-      <material name="eye_white"/></visual>
+      <xacro:m_eye_white/></visual>
     <!-- Left iris -->
     <visual><origin xyz="0.038 0.108 0.14" rpy="-1.5708 0 0"/>
       <geometry><cylinder radius="0.010" length="0.004"/></geometry>
-      <material name="eye_iris"/></visual>
+      <xacro:m_eye_iris/></visual>
     <!-- Right iris -->
     <visual><origin xyz="-0.038 0.108 0.14" rpy="-1.5708 0 0"/>
       <geometry><cylinder radius="0.010" length="0.004"/></geometry>
-      <material name="eye_iris"/></visual>
+      <xacro:m_eye_iris/></visual>
     <!-- Mouth -->
     <visual><origin xyz="0 0.107 0.085" rpy="0 0 0"/>
       <geometry><box size="0.052 0.004 0.010"/></geometry>
-      <material name="mouth_red"/></visual>
+      <xacro:m_mouth_red/></visual>
     <collision><origin xyz="0 0 0.11" rpy="0 0 0"/>
       <geometry><sphere radius="0.11"/></geometry></collision>
@@ -337,9 +349,9 @@
     <visual><origin xyz="0 0 0" rpy="0 0 0"/>
       <geometry><sphere radius="0.045"/></geometry>
-      <material name="body_skin"/></visual>
+      <xacro:m_body_skin/></visual>
     <!-- Arm cylinder — extends -Z from shoulder -->
     <visual><origin xyz="0 0 -0.13" rpy="0 0 0"/>
       <geometry><cylinder radius="0.038" length="0.26"/></geometry>
-      <material name="body_skin"/></visual>
+      <xacro:m_body_skin/></visual>
     <collision><origin xyz="0 0 -0.13" rpy="0 0 0"/>
       <geometry><cylinder radius="0.038" length="0.26"/></geometry></collision>
@@ -370,10 +382,10 @@
     <visual><origin xyz="0 0 0" rpy="0 0 0"/>
       <geometry><sphere radius="0.032"/></geometry>
-      <material name="body_skin"/></visual>
+      <xacro:m_body_skin/></visual>
     <!-- Forearm cylinder -->
     <visual><origin xyz="0 0 -0.11" rpy="0 0 0">
       </origin>
       <geometry><cylinder radius="0.032" length="0.22"/></geometry>
-      <material name="body_skin"/></visual>
+      <xacro:m_body_skin/></visual>
     <collision><origin xyz="0 0 -0.11" rpy="0 0 0">
       </origin>
@@ -392,5 +404,5 @@
     <visual><origin xyz="0 0 -0.015" rpy="0 0 0"/>
       <geometry><box size="0.042 0.052 0.030"/></geometry>
-      <material name="body_skin"/></visual>
+      <xacro:m_body_skin/></visual>
     <collision><origin xyz="0 0 -0.015" rpy="0 0 0">
       </origin>
@@ -422,9 +434,9 @@
       </origin>
       <geometry><sphere radius="0.045"/></geometry>
-      <material name="body_skin"/></visual>
+      <xacro:m_body_skin/></visual>
     <visual><origin xyz="0 0 -0.13" rpy="0 0 0">
       </origin>
       <geometry><cylinder radius="0.038" length="0.26"/></geometry>
-      <material name="body_skin"/></visual>
+      <xacro:m_body_skin/></visual>
     <collision><origin xyz="0 0 -0.13" rpy="0 0 0">
       </origin>
@@ -455,9 +467,9 @@
       </origin>
       <geometry><sphere radius="0.032"/></geometry>
-      <material name="body_skin"/></visual>
+      <xacro:m_body_skin/></visual>
     <visual><origin xyz="0 0 -0.11" rpy="0 0 0">
       </origin>
       <geometry><cylinder radius="0.032" length="0.22"/></geometry>
-      <material name="body_skin"/></visual>
+      <xacro:m_body_skin/></visual>
     <collision><origin xyz="0 0 -0.11" rpy="0 0 0">
       </origin>
@@ -477,5 +489,5 @@
       </origin>
       <geometry><box size="0.042 0.052 0.030"/></geometry>
-      <material name="body_skin"/></visual>
+      <xacro:m_body_skin/></visual>
     <collision><origin xyz="0 0 -0.015" rpy="0 0 0">
       </origin>
@@ -514,10 +526,10 @@
       </origin>
       <geometry><sphere radius="0.048"/></geometry>
-      <material name="body_dark"/></visual>
+      <xacro:m_body_dark/></visual>
     <!-- Thigh cylinder -->
     <visual><origin xyz="0 0 -0.14" rpy="0 0 0">
       </origin>
       <geometry><cylinder radius="0.048" length="0.28"/></geometry>
-      <material name="body_dark"/></visual>
+      <xacro:m_body_dark/></visual>
     <collision><origin xyz="0 0 -0.14" rpy="0 0 0">
       </origin>
@@ -536,10 +548,10 @@
       </origin>
       <geometry><sphere radius="0.038"/></geometry>
-      <material name="body_skin"/></visual>
+      <xacro:m_body_skin/></visual>
     <!-- Shin cylinder -->
     <visual><origin xyz="0 0 -0.145" rpy="0 0 0">
       </origin>
       <geometry><cylinder radius="0.036" length="0.29"/></geometry>
-      <material name="body_dark"/></visual>
+      <xacro:m_body_dark/></visual>
     <collision><origin xyz="0 0 -0.145" rpy="0 0 0">
       </origin>
@@ -557,5 +569,5 @@
       </origin>
       <geometry><box size="0.09 0.10 0.06"/></geometry>
-      <material name="body_dark"/></visual>
+      <xacro:m_body_dark/></visual>
     <collision><origin xyz="0 0.04 -0.03" rpy="0 0 0">
       </origin>
@@ -585,9 +597,9 @@
       </origin>
       <geometry><sphere radius="0.048"/></geometry>
-      <material name="body_dark"/></visual>
+      <xacro:m_body_dark/></visual>
     <visual><origin xyz="0 0 -0.14" rpy="0 0 0">
       </origin>
       <geometry><cylinder radius="0.048" length="0.28"/></geometry>
-      <material name="body_dark"/></visual>
+      <xacro:m_body_dark/></visual>
     <collision><origin xyz="0 0 -0.14" rpy="0 0 0">
       </origin>
@@ -605,9 +617,9 @@
       </origin>
       <geometry><sphere radius="0.038"/></geometry>
-      <material name="body_skin"/></visual>
+      <xacro:m_body_skin/></visual>
     <visual><origin xyz="0 0 -0.145" rpy="0 0 0">
       </origin>
       <geometry><cylinder radius="0.036" length="0.29"/></geometry>
-      <material name="body_dark"/></visual>
+      <xacro:m_body_dark/></visual>
     <collision><origin xyz="0 0 -0.145" rpy="0 0 0">
       </origin>
@@ -625,5 +637,5 @@
       </origin>
       <geometry><box size="0.09 0.10 0.06"/></geometry>
-      <material name="body_dark"/></visual>
+      <xacro:m_body_dark/></visual>
     <collision><origin xyz="0 0.04 -0.03" rpy="0 0 0">
       </origin>
